Commit message: Add files via upload

File: generar_URDF/urdf/macro_joints.xacro (robot description, xacro)
@@ -1,6 +1,10 @@
 <?xml version="1.0"?>
 <robot name="box_bot" xmlns:xacro="http://www.ros.org/wiki/xacro">
+<xacro:arg name="px1" default="1"/>
+<xacro:arg name="pz2" default="1"/>
+<xacro:arg name="n_90_grad2" default="1"/>
+<xacro:property name="n_90_grad2" value="$(arg n_90_grad2)"/> <!-- Se pasa a propiedad para poder hacer cálculos con ella -->
 <xacro:property name="angulo_recto" value="${pi/2}"/>
-<xacro:macro name="create_link" params="name xyz:=0 0 0 rpy:= 0 0 0">
+<xacro:macro name="create_link" params="name xyz:='0 0 0' rpy:= '0 0 0'">
   <link name="${name}">
     <visual>
@@ -26,5 +30,5 @@
   </link>
 </xacro:macro>
-<xacro:macro name="create_joint" params="name parent child xyz:= 0 0 0 rpy:= 0 0 0">
+<xacro:macro name="create_joint" params="name parent child xyz:= '0 0 0' rpy:= '0 0 0'">
   <joint name="${name}" type="fixed">
     <parent link="${parent}"/>
@@ -34,7 +38,7 @@
 </xacro:macro>
 <xacro:create_link name="base_link"/>
-<xacro:create_joint name="joint1" parent="base_link" child="link1" xyz="1 0 0"/>
+<xacro:create_joint name="joint1" parent="base_link" child="link1" xyz="$(arg px1) 0 0"/>
 <xacro:create_link name="link1"/>
-<xacro:create_joint name="joint2" parent="link1" child="link2" xyz="0 0 1" rpy="0 0 ${angulo_recto}"/>
+<xacro:create_joint name="joint2" parent="link1" child="link2" xyz="0 0 $(arg pz2)" rpy="0 0 ${angulo_recto*n_90_grad2}"/>
 <xacro:create_link name="link2"/>
 </robot>

File: generar_URDF/urdf/macro_links.xacro (robot description, xacro)
@@ -1,4 +1,8 @@
 <?xml version="1.0"?>
 <robot name="box_bot" xmlns:xacro="http://www.ros.org/wiki/xacro">
+<xacro:arg name="px1" default="1"/>
+<xacro:arg name="pz2" default="1"/>
+<xacro:arg name="n_90_grad2" default="1"/>
+<xacro:property name="n_90_grad2" value="$(arg n_90_grad2)"/> <!-- Se pasa a propiedad para poder hacer cálculos con ella -->
 <xacro:property name="angulo_recto" value="${pi/2}"/>
 <xacro:macro name="create_link" params="name xyz:='0 0 0' rpy:='0 0 0'">
@@ -33,8 +37,8 @@
   </joint>
 </xacro:macro>
-<xacro:create_link name="base_link" xyz="1 0 0"/>
+<xacro:create_link name="base_link" xyz="$(arg px1) 0 0"/>
 <xacro:create_joint name="joint1" parent="base_link" child="link1"/>
-<xacro:create_link name="link1" rpy="0 0 ${angulo_recto}"/>
+<xacro:create_link name="link1" rpy="0 0 ${angulo_recto*n_90_grad2}"/>
 <xacro:create_joint name="joint2" parent="link1" child="link2" />
-<xacro:create_link name="link2" xyz="0 0 1"/>
+<xacro:create_link name="link2" xyz="0 0 $(arg pz2)"/>
 </robot>

File: generar_URDF/urdf/model_joints.xacro (robot description, xacro)
@@ -26,5 +26,5 @@
   <parent link="base_link"/>
   <child link="link1"/>
-  <origin xyz="1 0 0" rpy="0 0 0"/> <!--0 0 1.57-->
+  <origin xyz="1 0 0" rpy="0 0 0"/>
 </joint>
 <link name="link1">
